File: Flight_Computer.sch (KiCad schematic (older format))
At the start: 43 parts, among them IC1 PIC32MZ2048EFH144-I_PL, J1 ICSP Programming, J2 Stack Connector, U1 STMPS2141STR, U2 STMPS2141STR, U3 BNO055

Commit message: Added SD card, CAN interface, many more updates. Also introduced PCB Template
Parts:
- removed J2: Stack Connector, symbol Connector_Generic:Conn_02x20_Odd_Even
- added C21, C24, C25: 100p, Capacitor_SMD:C_0603_1608Metric, symbol Device:C_Small
- added C22, C? (x4): 1n, Capacitor_SMD:C_0603_1608Metric, symbol Device:C_Small
- added C23, C26, C?: 100n, Capacitor_SMD:C_0603_1608Metric, symbol Device:C_Small
- added D3: D_TVS_x2_AAC, Package_TO_SOT_SMD:SOT-23, symbol Device:D_TVS_x2_AAC
- added J1: SC_19-20, MASA_Library:Stack_Connector_2019_2020, symbol MASA_Library:SC_19-20
- added J4: 47219-2001, 472192001, symbol MASA_Library:47219-2001
- added R13, R14, R16: 0, Resistor_SMD:R_0603_1608Metric, symbol Device:R_Small_US
- added R15, R?: 10k, Resistor_SMD:R_0603_1608Metric, symbol Device:R_Small_US
- added R17, R18: 60, Resistor_SMD:R_0603_1608Metric, symbol Device:R_Small_US
- added TP? (x10): T, symbol Connector:TestPoint
- added U4: SN65HVD1050D, Package_SO:SOIC-8_3.9x4.9mm_P1.27mm, symbol Interface_CAN_LIN:SN65HVD1050D
- added U?: TXB0104PWR, digikey-footprints:TSSOP-14_W4.4mm, symbol dk_Logic-Translators-Level-Shifters:TXB0104PWR
- C11, C12: footprint (none) -> Capacitor_SMD:CP_Elec_5x3
- D1, D2: footprint (none) -> Diode_SMD:D_0805_2012Metric
- J3: renamed from J1; footprint (none) -> Connector_PinHeader_2.54mm:PinHeader_1x05_P2.54mm_Vertical
- L1, L2: footprint (none) -> Inductor_SMD:L_Bourns-SRN4018
- gave numbers to parts that had none: 3
Connections:
- net labels added: +3.3V, CAN_H, CAN_L, CAN_RX, CAN_TX, SD_CLK, SD_CLK_L, SD_CS, SD_CS_L, SD_MISO, SD_MISO_L, SD_MOSI, SD_MOSI_L
- wire segments 126 -> 188
- no-connect marks 2 -> 4
Other:
- note removed: "Stack Connector\n"
- moved on the sheet: C18, C19, C20, R11, R12, U3

Commit message: Many changes
Parts:
- removed R11: 10k, Resistor_SMD:R_0805_2012Metric, symbol Device:R_Small_US
- added C19, C24, C25, C44, C45, C46, C53: 1n, Capacitor_SMD:C_0402_1005Metric, symbol Device:C_Small
- added C21, C22, C23, C26, C27: 100n, Capacitor_SMD:C_0402_1005Metric, symbol Device:C_Small
- added C28, C29: 2.2u, Capacitor_SMD:C_0402_1005Metric, symbol Device:C_Small
- added C34: 1n, Capacitor_SMD:C_0603_1608Metric, symbol Device:C_Small
- added C35, C54, C55: 100n, Capacitor_SMD:C_0603_1608Metric, symbol Device:C_Small
- added C47, C48, C49: 10n, Capacitor_SMD:C_0402_1005Metric, symbol Device:C_Small
- added C50, C51, C52: 1u, Capacitor_SMD:C_0402_1005Metric, symbol Device:C_Small
- added L3, L4: 2.2u, Inductor_SMD:L_0402_1005Metric, symbol Device:L
- added L5, L6, L7: 220n, Inductor_SMD:L_0402_1005Metric, symbol Device:L
- added Q1, Q2: Q_NPN_BCE, Package_TO_SOT_SMD:SOT-23, symbol Device:Q_NPN_BCE
- added R12, R25: 1k, Resistor_SMD:R_0402_1005Metric, symbol Device:R_Small_US
- added R13, R14, R22, R23, R24: 3.3, Resistor_SMD:R_0402_1005Metric, symbol Device:R_Small_US
- added R26, R27: 10k, Resistor_SMD:R_0402_1005Metric, symbol Device:R_Small_US
- added TMP1, TMP2: LM50CIM3X, Package_TO_SOT_SMD:SOT-23, symbol MASA_Library:LM50CIM3X
- C14: renamed from C9; value 18u -> 22u
- C15: renamed from C10; value 18u -> 22u
- C16: renamed from C11; footprint Capacitor_SMD:CP_Elec_5x3 -> Capacitor_SMD:CP_Elec_5x5.3
- C17: renamed from C12; footprint Capacitor_SMD:CP_Elec_5x3 -> Capacitor_SMD:CP_Elec_5x5.3
- C18: renamed from C23; footprint Capacitor_SMD:C_0603_1608Metric -> Capacitor_SMD:C_0402_1005Metric
- C20: renamed from C22; footprint Capacitor_SMD:C_0603_1608Metric -> Capacitor_SMD:C_0402_1005Metric
- C36, C37, C38, C42, C43: renamed from C?; footprint Capacitor_SMD:C_0603_1608Metric -> Capacitor_SMD:C_0402_1005Metric
- L1: value 9.1u -> 3.3u; footprint Inductor_SMD:L_Bourns-SRN4018 -> Inductor_SMD:L_Wuerth_MAPI-2512; DK_Detail_Page (none) -> https://www.digikey.com/product-detail/en/w-rth-elektronik/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; Digi-Key_PN (none) -> 732-5684-1-ND; MPN (none) -> 74438324033; PART# (none) -> 74438324033
- L2: value 9.1u -> 3.3u; footprint Inductor_SMD:L_Bourns-SRN4018 -> Inductor_SMD:L_Wuerth_MAPI-2512; DK_Detail_Page (none) -> https://www.digikey.com/product-detail/en/w-rth-elektronik/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; Digi-Key_PN (none) -> 732-5684-1-ND; MPN (none) -> 74438324033
- R10, R9: value 700m -> 470m
- R21: renamed from R?; footprint Resistor_SMD:R_0603_1608Metric -> Resistor_SMD:R_0402_1005Metric
- TP1, TP10, TP2, TP3, TP4, TP5, TP6, TP7, TP8, TP9: renamed from TP?; footprint (none) -> TestPoint:TestPoint_Pad_1.0x1.0mm
- gave numbers to parts that had none: 1
- renumbered C16 to C10, C17 to C11, C5 to C12, C6 to C13, C18 to C30, C19 to C31, C21 to C32, C20 to C33, C24 to C39, C25 to C40, C26 to C41, C7 to C5, C8 to C6, C13 to C7, C14 to C8, C15 to C9, J3 to J1, J1 to J2, J2 to J3, R12 to R11, R13 to R15, R14 to R16, R15 to R17, R16 to R18, R17 to R19, R18 to R20, R7 to R3, R8 to R4, R3 to R5, R4 to R6, R5 to R7, R6 to R8
Connections:
- net +3V3: no longer U5.14 (VCCB)
- net +5V: now also C19.1, C21.1, C34.2, C35.2, R26.2, R27.2, TMP1.1 (Vs), TMP2.1 (Vs)
- net BNO_RX: now also IC1.91 (EBIA8/RPF5/SCL5/PMA8/RF5)
- net BNO_TX: now also IC1.90 (EBIA9/RPF4/SDA5/PMA9/RF4)
- net CAN_H: now also J2.21 (CAN_H)
- net CAN_L: now also J2.23 (CAN_L)
- net GND: now also C19.2, C21.2, C22.1, C23.1, C24.1, C25.1, C26.1, C27.1, C34.1, C35.1, C44.1, C45.1, C46.1, C47.1, C48.1, C49.1, C53.1, C54.2, C55.2, Q1.3 (E), Q2.3 (E), R13.2, R14.2, R22.2, R23.2, R24.2, TMP1.3 (GND), TMP2.3 (GND)
- net SD_CLK: now also C49.2, C52.2, L7.2
- net SD_CS: now also C53.2
- net SD_MISO: now also C48.2, C51.2, L6.2
- net SD_MOSI: now also C47.2, C50.2, L5.2
- net SCK: now reaches IC1.109 (RPD1/SCK1/RD1)
- net SCK: now also C46.2, L7.1
- net SDO: now reaches IC1.110 (EBID14/RPD2/PMD14/RD2)
- net SDO: now also C44.2, L5.1
- net SDI: now reaches IC1.120 (ETXEN/RPD6/RD6)
- net SDI1: now reaches IC1.97 (EBIA15/RPD9/PMCS2/PMA15/RD9)
- net SDI1: now also C45.2, L6.1
- net UART1_TX: now reaches J2.25 (UART1_TX)
- net UART1_RX: now reaches J2.27 (UART1_RX)
- net UART2_TX: now reaches J2.29 (UART2_TX)
- net UART2_RX: now reaches J2.31 (UART2_RX)
- net !BNO_BL_LOAD: no longer names the net of R11.1, U3.4 (BOOT_LOAD)
- net !BNO_BL_LOAD: now also Q1.2 (C), R26.1
- net !BNO_ENABLE: no longer names the net of U3.11 (RESET)
- net !BNO_ENABLE: now also Q2.2 (C), R27.1
- new net: C29.1, R14.1
- new net: C23.2, C25.2, L4.1, TMP2.2 (Vout)
- new net: C50.1, R22.1
- new net: C51.1, R23.1
- new net: C52.1, R24.1
- new net: C22.2, C24.2, L3.1, TMP1.2 (Vout)
- new net: C54.1, Q1.1 (B), R12.1
- new net: C55.1, Q2.1 (B), R25.1
- new net: C28.1, R13.1
- new net BNO_BL_LOAD: R12.2
- new net BNO_ENABLE: R25.2
- new net TSENSE_1: C26.2, C27.2, C28.2, C29.2, L3.2, L4.2
Other:
- moved on the sheet: C11, C18, C20, C3, C30, C31, C32, C33, C36, C37, C38, C39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
