File: Flight_Computer.kicad_pcb (KiCad board)
At the start: 4 copper layers, 75.8 x 76.2 mm, 58 parts, among them IC1 PIC32MZ2048EFH144-I_PL, J1 SC_19-20, J2 UJ2-MBH-1-SMT-TR, J3 ICSP Programming, J4 47219-2001, U1 STMPS2141STR, U2 STMPS2141STR, U3 BNO055, U4 SN65HVD1050D

Commit message: Many changes
Parts:
- removed the R11 at (245.5, 121.3)
- added C19: 1n, Capacitor_SMD:C_0402_1005Metric, F.Cu at (213.4, 74.9)
- added C21: 100n, Capacitor_SMD:C_0402_1005Metric, F.Cu at (219.0, 80.9)
- added C22: 100n, Capacitor_SMD:C_0402_1005Metric, F.Cu at (215.0, 84.9)
- added C23: 100n, Capacitor_SMD:C_0402_1005Metric, F.Cu at (213.9, 87.0)
- added C24: 1n, Capacitor_SMD:C_0402_1005Metric, F.Cu at (210.4, 78.9)
- added C25: 1n, Capacitor_SMD:C_0402_1005Metric, F.Cu at (217.9, 84.9)
- added C26: 100n, Capacitor_SMD:C_0402_1005Metric, F.Cu at (216.8, 86.9)
- added C27: 100n, Capacitor_SMD:C_0402_1005Metric, F.Cu at (220.8, 82.9)
- added C28: 2.2u, Capacitor_SMD:C_0402_1005Metric, F.Cu at (220.8, 84.9)
- added C29: 2.2u, Capacitor_SMD:C_0402_1005Metric, F.Cu at (211.0, 87.0)
- added C34: 1n, Capacitor_SMD:C_0603_1608Metric, F.Cu at (196.9, 83.4)
- added C35: 100n, Capacitor_SMD:C_0603_1608Metric, F.Cu at (200.9, 79.2)
- added C36: 100n, Capacitor_SMD:C_0402_1005Metric, F.Cu at (207.4, 81.0)
- added C37: 1n, Capacitor_SMD:C_0402_1005Metric, F.Cu at (216.5, 71.9)
- added C38: 1n, Capacitor_SMD:C_0402_1005Metric, F.Cu at (203.4, 84.5)
- added C42: 1n, Capacitor_SMD:C_0402_1005Metric, F.Cu at (215.0, 82.9)
- added C43: 1n, Capacitor_SMD:C_0402_1005Metric, F.Cu at (210.4, 76.9)
- added C44: 1n, Capacitor_SMD:C_0402_1005Metric, F.Cu at (210.4, 74.9)
- added C45: 1n, Capacitor_SMD:C_0402_1005Metric, F.Cu at (203.4, 82.5)
- added C46: 1n, Capacitor_SMD:C_0402_1005Metric, F.Cu at (213.4, 76.9)
- added C47: 10n, Capacitor_SMD:C_0402_1005Metric, F.Cu at (216.3, 74.9)
- added C48: 10n, Capacitor_SMD:C_0402_1005Metric, F.Cu at (206.3, 83.0)
- added C49: 10n, Capacitor_SMD:C_0402_1005Metric, F.Cu at (219.4, 71.9)
- added C50: 1u, Capacitor_SMD:C_0402_1005Metric, F.Cu at (210.3, 81.0)
- added C51: 1u, Capacitor_SMD:C_0402_1005Metric, F.Cu at (206.3, 85.0)
- added C52: 1u, Capacitor_SMD:C_0402_1005Metric, F.Cu at (205.2, 87.0)
- added C53: 1n, Capacitor_SMD:C_0402_1005Metric, F.Cu at (209.2, 83.0)
- added C54: 100n, Capacitor_SMD:C_0603_1608Metric, F.Cu at (196.9, 80.9)
- added C55: 100n, Capacitor_SMD:C_0603_1608Metric, F.Cu at (199.0, 76.7)
- added L3: 2.2u, Inductor_SMD:L_0402_1005Metric, F.Cu at (216.3, 78.9)
- added L4: 2.2u, Inductor_SMD:L_0402_1005Metric, F.Cu at (213.4, 78.9)
- added L5: 220n, Inductor_SMD:L_0402_1005Metric, F.Cu at (202.3, 87.5)
- added L6: 220n, Inductor_SMD:L_0402_1005Metric, F.Cu at (199.4, 87.5)
- added L7: 220n, Inductor_SMD:L_0402_1005Metric, F.Cu at (219.2, 73.9)
- added Q1: Q_NPN_BCE, Package_TO_SOT_SMD:SOT-23, F.Cu at (192.7, 81.9)
- added Q2: Q_NPN_BCE, Package_TO_SOT_SMD:SOT-23, F.Cu at (199.2, 73.2)
- added R12: 1k, Resistor_SMD:R_0402_1005Metric, F.Cu at (219.2, 77.8)
- added R13: 3.3, Resistor_SMD:R_0402_1005Metric, F.Cu at (212.1, 85.0)
- added R14: 3.3, Resistor_SMD:R_0402_1005Metric, F.Cu at (217.9, 82.9)
- added R21: 10k, Resistor_SMD:R_0402_1005Metric, F.Cu at (213.2, 80.9)
- added R22: 3.3, Resistor_SMD:R_0402_1005Metric, F.Cu at (209.2, 85.0)
- added R23: 3.3, Resistor_SMD:R_0402_1005Metric, F.Cu at (208.1, 87.0)
- added R24: 3.3, Resistor_SMD:R_0402_1005Metric, F.Cu at (219.2, 75.9)
- added R25: 1k, Resistor_SMD:R_0402_1005Metric, F.Cu at (212.1, 83.0)
- added R26: 10k, Resistor_SMD:R_0402_1005Metric, F.Cu at (216.3, 76.9)
- added R27: 10k, Resistor_SMD:R_0402_1005Metric, F.Cu at (216.1, 80.9)
- added TMP1: LM50CIM3X, Package_TO_SOT_SMD:SOT-23, F.Cu at (203.7, 73.2)
- added TMP2: LM50CIM3X, Package_TO_SOT_SMD:SOT-23, F.Cu at (192.7, 86.5)
- added TP1: T, TestPoint:TestPoint_Pad_1.0x1.0mm, F.Cu at (207.4, 72.4)
- added TP10: T, TestPoint:TestPoint_Pad_1.0x1.0mm, F.Cu at (200.4, 82.0)
- added TP2: T, TestPoint:TestPoint_Pad_1.0x1.0mm, F.Cu at (207.5, 78.5)
- added TP3: T, TestPoint:TestPoint_Pad_1.0x1.0mm, F.Cu at (213.5, 72.4)
- added TP4: T, TestPoint:TestPoint_Pad_1.0x1.0mm, F.Cu at (204.4, 80.0)
- added TP5: T, TestPoint:TestPoint_Pad_1.0x1.0mm, F.Cu at (207.5, 75.5)
- added TP6: T, TestPoint:TestPoint_Pad_1.0x1.0mm, F.Cu at (200.4, 85.0)
- added TP7: T, TestPoint:TestPoint_Pad_1.0x1.0mm, F.Cu at (196.4, 86.2)
- added TP8: T, TestPoint:TestPoint_Pad_1.0x1.0mm, F.Cu at (210.4, 72.4)
- added TP9: T, TestPoint:TestPoint_Pad_1.0x1.0mm, F.Cu at (204.4, 77.0)
- added U5: TXB0104PWR, digikey-footprints:TSSOP-14_W4.4mm, F.Cu at (193.7, 75.3)
- C14: renamed from C9; value 18u -> 22u
- C15: renamed from C10; value 18u -> 22u
- C16: renamed from C11; footprint Capacitor_SMD:CP_Elec_5x3 -> Capacitor_SMD:CP_Elec_5x5.3
- C17: renamed from C12; footprint Capacitor_SMD:CP_Elec_5x3 -> Capacitor_SMD:CP_Elec_5x5.3
- C18: renamed from C23; footprint Capacitor_SMD:C_0603_1608Metric -> Capacitor_SMD:C_0402_1005Metric
- C20: renamed from C22; footprint Capacitor_SMD:C_0603_1608Metric -> Capacitor_SMD:C_0402_1005Metric
- L1, L2: value 9.1u -> 3.3u; footprint Inductor_SMD:L_Bourns-SRN4018 -> Inductor_SMD:L_Wuerth_MAPI-2512
- R10, R9: value 700m -> 470m
- renumbered C16 to C10, C17 to C11, C5 to C12, C6 to C13, C18 to C30, C19 to C31, C21 to C32, C20 to C33, C24 to C39, C25 to C40, C26 to C41, C7 to C5, C8 to C6, C13 to C7, C14 to C8, C15 to C9, J3 to J1, J1 to J2, J2 to J3, R12 to R11, R13 to R15, R14 to R16, R15 to R17, R16 to R18, R17 to R19, R18 to R20, R7 to R3, R8 to R4, R3 to R5, R4 to R6, R5 to R7, R6 to R8
Connections:
- net !BNO_BL_LOAD renamed Net-(Q1-Pad2)
- net Net-(IC1-Pad120) renamed SDI
- net Net-(J1-Pad25) renamed UART1_TX
- net Net-(J1-Pad27) renamed UART1_RX
- net Net-(J1-Pad29) renamed UART2_TX
- net Net-(J1-Pad31) renamed UART2_RX
- IC1 pad 109: Net-(IC1-Pad109) -> SCK
- IC1 pad 110: Net-(IC1-Pad110) -> SDO
- IC1 pad 90: Net-(IC1-Pad90) -> BNO_TX
- IC1 pad 91: Net-(IC1-Pad91) -> BNO_RX
- IC1 pad 97: Net-(IC1-Pad97) -> SDI1
- J2 pad 21: Net-(J1-Pad21) -> CAN_H
- J2 pad 23: Net-(J1-Pad23) -> CAN_L
- J4 pad 10: Net-(J4-Pad10) -> GND
- J4 pad 11: Net-(J4-Pad11) -> GND
- J4 pad 12: Net-(J4-Pad12) -> GND
- J4 pad 2: Net-(J4-Pad2) -> SD_CS_L
- J4 pad 3: Net-(J4-Pad3) -> SD_MOSI_L
- J4 pad 4: Net-(J4-Pad4) -> +3V3
- J4 pad 5: Net-(J4-Pad5) -> SD_CLK_L
- J4 pad 6: Net-(J4-Pad6) -> GND
- J4 pad 7: Net-(J4-Pad7) -> SD_MISO_L
- J4 pad 9: Net-(J4-Pad9) -> GND
- U3 pad 11: !BNO_ENABLE -> Net-(Q2-Pad2)

Commit message: Routing progress
Parts:
- removed C16, C17: 100u, Capacitor_SMD:CP_Elec_5x5.3
- removed C38, C42, C43, C53: 1n, Capacitor_SMD:C_0402_1005Metric
- removed R21: 10k, Resistor_SMD:R_0402_1005Metric
- removed U5: TXB0104PWR, digikey-footprints:TSSOP-14_W4.4mm
- added C56: 1u, Capacitor_SMD:C_0402_1005Metric, F.Cu at (220.0, 153.9)
- added C57: 1u, Capacitor_SMD:C_0402_1005Metric, F.Cu at (214.1, 153.9)
- added C58: 1u, Capacitor_SMD:C_0402_1005Metric, F.Cu at (225.0, 147.2)
- added C59: 1u, Capacitor_SMD:C_0402_1005Metric, F.Cu at (220.0, 151.9)
- added C60: 10n, Capacitor_SMD:C_0402_1005Metric, F.Cu at (217.1, 153.9)
- added C61: 10n, Capacitor_SMD:C_0402_1005Metric, F.Cu at (227.9, 143.2)
- added C62: 10n, Capacitor_SMD:C_0402_1005Metric, F.Cu at (214.1, 155.9)
- added C63: 10n, Capacitor_SMD:C_0402_1005Metric, F.Cu at (225.0, 145.2)
- added C64: 1n, Capacitor_SMD:C_0402_1005Metric, F.Cu at (217.1, 151.9)
- added C65: 1n, Capacitor_SMD:C_0402_1005Metric, F.Cu at (205.3, 154.9)
- added C66: 1n, Capacitor_SMD:C_0402_1005Metric, F.Cu at (225.0, 143.2)
- added C67: 1n, Capacitor_SMD:C_0402_1005Metric, F.Cu at (211.1, 154.9)
- added C68: 1n, Capacitor_SMD:C_0402_1005Metric, F.Cu at (151.4, 93.5)
- added C69: 1n, Capacitor_SMD:C_0402_1005Metric, F.Cu at (160.0, 100.6)
- added C70: 1n, Capacitor_SMD:C_0402_1005Metric, F.Cu at (155.4, 100.6)
- added IC2: FAN4010IL6X_F113, MASA_Library:6-LEAD_MICROPAK, F.Cu at (145.4, 114.3)
- added IC3: FAN4010IL6X_F113, MASA_Library:6-LEAD_MICROPAK, F.Cu at (173.3, 116.4)
- added L10: 220n, Inductor_SMD:L_0402_1005Metric, F.Cu at (222.8, 155.9)
- added L11: 220n, Inductor_SMD:L_0402_1005Metric, F.Cu at (227.9, 149.2)
- added L8: 220n, Inductor_SMD:L_0402_1005Metric, F.Cu at (228.7, 151.1)
- added L9: 220n, Inductor_SMD:L_0402_1005Metric, F.Cu at (225.8, 153.1)
- added R28: 3.3, Resistor_SMD:R_0402_1005Metric, F.Cu at (222.9, 153.9)
- added R29: 3.3, Resistor_SMD:R_0402_1005Metric, F.Cu at (219.9, 155.9)
- added R30: 3.3, Resistor_SMD:R_0402_1005Metric, F.Cu at (227.9, 147.2)
- added R31: 10k, Resistor_SMD:R_0402_1005Metric, F.Cu at (153.9, 93.5)
- added R32: 3.3k, Resistor_SMD:R_0402_1005Metric, F.Cu at (148.3, 114.7)
- added R33: 3.3k, Resistor_SMD:R_0402_1005Metric, F.Cu at (173.0, 118.5)
- added R34: 220m, Resistor_SMD:R_0805_2012Metric, F.Cu at (145.4, 116.6)
- added R35: 220m, Resistor_SMD:R_0805_2012Metric, F.Cu at (173.2, 114.7)
- added U8: TXB0104PWR, digikey-footprints:TSSOP-14_W4.4mm, F.Cu at (157.7, 97.1)
- C12, C13: value 1n -> 100n; footprint Capacitor_SMD:C_0805_2012Metric -> Capacitor_SMD:C_0402_1005Metric
- C32, C34, C35, C39, C40, C41, C54, C55: footprint Capacitor_SMD:C_0603_1608Metric -> Capacitor_SMD:C_0402_1005Metric
- L1: value 3.3u -> 4.7u; footprint Inductor_SMD:L_Wuerth_MAPI-2512 -> Capacitor_SMD:C_0805_2012Metric
- L2: value 3.3u -> 4.7u; footprint Inductor_SMD:L_Wuerth_MAPI-2512 -> Inductor_SMD:L_0805_2012Metric
- Q1, Q2: value Q_NPN_BCE -> Q_NPN_BEC
- R10, R9: value 470m -> 1; footprint Resistor_SMD:R_0805_2012Metric -> Resistor_SMD:R_0402_1005Metric
- R11: value 10k -> 3.3; footprint Resistor_SMD:R_0805_2012Metric -> Resistor_SMD:R_0402_1005Metric
- R5, R6, R7, R8: footprint Resistor_SMD:R_0805_2012Metric -> Resistor_SMD:R_0402_1005Metric
- moved C14 110.2 mm to (149.1, 116.6)
- moved U1 102.5 mm to (141.2, 118.8), turned to 90 degrees
- moved C12 99.1 mm to (142.0, 121.4), turned to 180 degrees
- moved TP10 98.9 mm to (273.8, 148.3)
- moved R7 97.7 mm to (140.3, 116.0), turned to 180 degrees
- moved TP9 97.3 mm to (273.8, 145.2)
- moved TP8 96.9 mm to (270.7, 148.3)
- moved R5 95.9 mm to (138.0, 118.4), turned to 90 degrees
- moved TP7 94.9 mm to (270.7, 145.2)
- moved R8 93.5 mm to (161.4, 119.9), turned to 90 degrees
- moved TP6 92.3 mm to (267.7, 148.3)
- moved TP5 92.2 mm to (267.7, 145.2)
- moved D1 91.9 mm to (144.8, 119.5), turned to 270 degrees
- moved R6 91.2 mm to (163.8, 117.4), turned to 180 degrees
- moved TP4 91.0 mm to (264.6, 148.3)
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Connections:
- C14 pad 1: +3V3 -> Net-(C14-Pad1)
- C14 pad 2: GND -> Net-(C14-Pad2)
- C15 pad 1: +5V -> Net-(C15-Pad1)
- C15 pad 2: GND -> Net-(C15-Pad2)
- C27 pad 2: TSENSE_1 -> TSENSE_2
- C29 pad 2: TSENSE_1 -> TSENSE_2
- IC1 pad 100: Net-(IC1-Pad100) -> BNO_ENABLE
- IC1 pad 101: Net-(IC1-Pad101) -> BNO_BL_LOAD
- IC1 pad 102: Net-(IC1-Pad102) -> BNO_BL_IND
- IC1 pad 103: Net-(IC1-Pad103) -> BNO_INT
- IC1 pad 118: Net-(IC1-Pad118) -> UART1_RX
- IC1 pad 119: Net-(IC1-Pad119) -> UART1_TX
- IC1 pad 127: Net-(IC1-Pad127) -> UART2_TX
- IC1 pad 128: Net-(IC1-Pad128) -> UART2_RX
- IC1 pad 49: Net-(IC1-Pad49) -> TSENSE_1
- IC1 pad 50: Net-(IC1-Pad50) -> TSENSE_2
- IC1 pad 65: Net-(IC1-Pad65) -> I_5V
- IC1 pad 66: Net-(IC1-Pad66) -> I_3V3
- J2 pad 25: UART1_TX -> Net-(C64-Pad2)
- J2 pad 27: UART1_RX -> Net-(C65-Pad2)
- J2 pad 29: UART2_TX -> Net-(C66-Pad2)
- J2 pad 31: UART2_RX -> Net-(C67-Pad2)
- J4 pad 2: SD_CS_L -> SD_CS
- J4 pad 3: SD_MOSI_L -> SD_MISO
- J4 pad 5: SD_CLK_L -> SD_CLK
- J4 pad 7: SD_MISO_L -> SD_MISO
- L1 pad 2: +3V3 -> Net-(C14-Pad1)
- L2 pad 2: +5V -> Net-(C15-Pad1)
- L4 pad 2: TSENSE_1 -> TSENSE_2
- Q1 pad 2: Net-(Q1-Pad2) -> GND
- Q1 pad 3: GND -> Net-(Q1-Pad3)
- Q2 pad 2: Net-(Q2-Pad2) -> GND
- Q2 pad 3: GND -> Net-(Q2-Pad3)
- R10 pad 2: Net-(C17-Pad2) -> Net-(C15-Pad2)
- R11 pad 1: Net-(Q1-Pad2) -> Net-(C56-Pad1)
- R11 pad 2: +5V -> GND
- R26 pad 1: Net-(Q1-Pad2) -> Net-(Q1-Pad3)
- R27 pad 1: Net-(Q2-Pad2) -> Net-(Q2-Pad3)
- R9 pad 2: Net-(C16-Pad2) -> Net-(C14-Pad2)
- TP5 pad 1: +3V3 -> Net-(C14-Pad1)
- TP6 pad 1: +5V -> Net-(C15-Pad1)
- U3 pad 11: Net-(Q2-Pad2) -> Net-(Q2-Pad3)
- U3 pad 19: BNO_RX -> Net-(U3-Pad19)
- U3 pad 20: BNO_TX -> Net-(U3-Pad20)
- U3 pad 4: Net-(Q1-Pad2) -> Net-(Q1-Pad3)
Routing:
- net +5V: track 0.00 -> 65.2 mm
- net GND: track 0.00 -> 30.3 mm, vias 0 -> 21
- net +3.3VP: track 0.00 -> 12.6 mm
- net +5VP: track 0.00 -> 10.9 mm
- net Net-(C13-Pad1): track 0.00 -> 7.22 mm
- net Net-(C15-Pad1): track 0.00 -> 7.08 mm
- net Net-(C12-Pad1): track 0.00 -> 6.94 mm
- net Net-(C14-Pad1): track 0.00 -> 6.27 mm
- net Net-(U3-Pad20): track 0.00 -> 5.29 mm
- net Net-(U3-Pad19): track 0.00 -> 5.21 mm
- net Net-(R6-Pad2): track 0.00 -> 3.87 mm
- net +3V3: track 0.00 -> 3.82 mm, vias 0 -> 3
- net Net-(R5-Pad2): track 0.00 -> 3.71 mm
- net Net-(C54-Pad1): track 0.00 -> 2.80 mm
- net Net-(Q1-Pad3): track 0.00 -> 2.78 mm
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- added copper zone on F.Cu, net +3V3
- added copper zone on In1.Cu, net +3V3
- added copper zone on B.Cu, net GND
Other:
- net class Default: clearance 0.254 -> 0.127; trace_width 0.254 -> 0.1524
- rule trace_clearance: 0.254 -> 0.127
- rule trace_min: 0.254 -> 0.1016

Commit message: More additions
Parts:
- R15, R16, R17, R18: footprint Resistor_SMD:R_0603_1608Metric -> Resistor_SMD:R_0402_1005Metric
- moved R16 99.3 mm to (166.0, 142.0)
- moved R19 99.1 mm to (164.3, 135.3)
- moved C32 92.8 mm to (170.4, 140.8), turned to 180 degrees
- moved R20 87.9 mm to (164.3, 133.6), turned to 180 degrees
- moved C41 84.8 mm to (166.6, 135.0), turned to 90 degrees
- moved U4 82.8 mm to (171.8, 136.2), turned to 90 degrees
- moved C39 80.2 mm to (162.1, 135.8), turned to 90 degrees
- moved R15 77.8 mm to (166.0, 140.9)
- moved C40 75.4 mm to (162.1, 133.2), turned to 90 degrees
- moved D3 74.1 mm to (153.7, 134.0), turned to 90 degrees
- moved R18 68.5 mm to (173.2, 131.2), turned to 180 degrees
- moved C35 68.4 mm to (172.1, 141.3), turned to 90 degrees
- moved R17 65.2 mm to (168.3, 138.8), turned to 90 degrees
- moved C34 62.5 mm to (173.3, 141.3), turned to 90 degrees
- moved L8 50.9 mm to (182.8, 129.0)
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Routing:
- net GND: track 30.3 -> 83.1 mm, vias 21 -> 44
- net CAN_H: track 0.00 -> 32.5 mm
- net CAN_L: track 0.00 -> 28.6 mm
- net USB_D+: track 0.00 -> 16.3 mm
- net USB_D-: track 0.00 -> 15.9 mm
- net USB_VBUS: track 0.00 -> 14.1 mm, vias 0 -> 2
- net Net-(C41-Pad2): track 0.00 -> 11.6 mm, vias 0 -> 2
- net +5V: track 65.2 -> 68.6 mm
- net Net-(R18-Pad1): track 0.00 -> 2.61 mm

Commit message: Finished routing
Parts:
- added R21: 3.3k, Resistor_SMD:R_0402_1005Metric, F.Cu at (127.8, 109.7)
- added R36: 3.3k, Resistor_SMD:R_0402_1005Metric, F.Cu at (181.1, 140.0)
- C1, C10, C11, C2, C3, C30, C31, C33, C4, C5, C6, C7, C8, C9: footprint Capacitor_SMD:C_0603_1608Metric -> Capacitor_SMD:C_0402_1005Metric
- R1, R2, R3, R4: footprint Resistor_SMD:R_0805_2012Metric -> Resistor_SMD:R_0402_1005Metric
- moved R2 128.6 mm to (138.9, 158.5)
- moved TP1 125.4 mm to (136.2, 148.1)
- moved C18 125.0 mm to (127.9, 104.8), turned to 180 degrees
- moved C20 123.0 mm to (127.9, 103.7), turned to 180 degrees
- moved TP2 122.7 mm to (138.9, 153.1)
- moved C5 120.8 mm to (145.9, 163.4)
- moved TP5 120.5 mm to (151.1, 114.7), turned to 270 degrees
- moved TP3 117.5 mm to (149.6, 121.1), turned to 270 degrees
- moved R4 116.5 mm to (137.4, 151.2), turned to 90 degrees
- moved C1 116.2 mm to (131.8, 149.8), turned to 270 degrees
- moved C6 115.6 mm to (147.4, 138.5)
- moved C30 114.2 mm to (144.0, 94.9), turned to 180 degrees
- moved C49 113.9 mm to (125.8, 136.8)
- moved C3 113.1 mm to (139.8, 150.1), turned to 90 degrees
- moved R3 112.0 mm to (137.9, 149.6)
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Connections:
- C1 pad 1: VDD -> +3V3
- C45 pad 2: SDI1 -> SD_MISO
- C48 pad 2: SD_MISO -> SDI
- C51 pad 2: SD_MISO -> SDI
- C56 pad 2: UART1_TX -> Net-(C56-Pad2)
- C58 pad 2: UART2_TX -> Net-(C58-Pad2)
- C60 pad 2: UART1_TX -> Net-(C56-Pad2)
- C62 pad 2: UART2_TX -> Net-(C58-Pad2)
- C64 pad 2: Net-(C64-Pad2) -> UART1_TX
- C66 pad 2: Net-(C66-Pad2) -> UART2_TX
- IC1 pad 97: SDI1 -> Net-(IC1-Pad97)
- J1 pad 2: VDD -> +3V3
- J2 pad 25: Net-(C64-Pad2) -> Net-(C56-Pad2)
- J2 pad 29: Net-(C66-Pad2) -> Net-(C58-Pad2)
- J4 pad 3: SD_MISO -> SD_MOSI
- L10 pad 1: Net-(C66-Pad2) -> UART2_TX
- L10 pad 2: UART2_TX -> Net-(C58-Pad2)
- L6 pad 1: SDI1 -> SD_MISO
- L6 pad 2: SD_MISO -> SDI
- L8 pad 1: Net-(C64-Pad2) -> UART1_TX
- L8 pad 2: UART1_TX -> Net-(C56-Pad2)
Routing:
- net GND: track 83.1 -> 183.6 mm, vias 44 -> 81
- net BNO_INT: track 0.00 -> 89.6 mm, vias 0 -> 2
- net BNO_BL_IND: track 0.00 -> 88.8 mm, vias 0 -> 2
- net I_3V3: track 2.37 -> 89.0 mm, vias 0 -> 2
- net BNO_BL_LOAD: track 0.00 -> 80.9 mm, vias 0 -> 2
- net TSENSE_1: track 0.00 -> 80.9 mm, vias 0 -> 2
- net BNO_ENABLE: track 0.00 -> 79.6 mm, vias 0 -> 2
- net BNO_RX: track 0.00 -> 77.7 mm, vias 0 -> 4
- net BNO_TX: track 0.00 -> 77.1 mm, vias 0 -> 4
- net I_5V: track 1.25 -> 63.2 mm, vias 0 -> 2
- net +5V: track 68.6 -> 128.5 mm, vias 0 -> 2
- net SD_MOSI: track 0.00 -> 48.8 mm, vias 0 -> 2
- net +3V3: track 3.82 -> 49.8 mm, vias 3 -> 14
- net TSENSE_2: track 0.00 -> 44.7 mm, vias 0 -> 2
- net SDI: track 0.00 -> 37.9 mm, vias 0 -> 2
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- added copper zone on F.Cu, net GND
- added copper zone on In2.Cu, net GND
