File: Flight_Computer.kicad_pcb (KiCad board)
At the start: 4 copper layers, 75.8 x 76.2 mm, 140 parts, among them IC1 PIC32MZ2048EFH144-I_PL, IC2 FAN4010IL6X_F113, IC3 FAN4010IL6X_F113, J1 ICSP Programming, J2 SC_19-20, J3 UJ2-MBH-1-SMT-TR, J4 47219-2001, Q1 Q_NPN_BEC, Q2 Q_NPN_BEC, U1 STMPS2141STR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

Commit message: Fixed CAN Bus voltage error
Parts:
- added U5: SN74LVC1T45DBVR, digikey-footprints:SOT-23-6, F.Cu at (178.9, 140.4)
- added U6: SN74LVC1T45DBVR, digikey-footprints:SOT-23-6, F.Cu at (178.9, 136.1)
- moved R16 8.94 mm to (174.9, 140.8), turned to 180 degrees
- moved R15 2.90 mm to (168.9, 141.3), turned to 90 degrees
- moved C21 2.14 mm to (183.2, 133.4)
- moved C25 2.14 mm to (183.6, 141.0)
- moved L4 2.14 mm to (182.5, 141.0)
- moved R36 2.14 mm to (183.2, 139.4)
- moved TMP2 2.14 mm to (183.7, 137.0)
- moved C29 2.14 mm to (183.1, 143.7)
- moved C19 2.14 mm to (183.2, 134.4)
- moved C23 2.14 mm to (184.7, 139.9)
- moved C27 2.14 mm to (183.1, 142.5)
- moved R14 2.14 mm to (184.7, 143.0)
- moved TP7 1.10 mm to (166.5, 140.8)
- moved TP8 0.79 mm to (166.6, 143.2)
Connections:
- R15 pad 1: CAN_TX -> Net-(R15-Pad1)
- R16 pad 1: CAN_RX -> Net-(R16-Pad1)
Routing:
- net CAN_RX: track 5.63 -> 30.0 mm
- net CAN_TX: track 6.18 -> 24.7 mm
- net +5V: track 128.5 -> 145.5 mm, vias 2 -> 5
- net Net-(R15-Pad1): track 0.00 -> 10.9 mm
- net Net-(R16-Pad2): track 11.8 -> 2.35 mm
- net Net-(R16-Pad1): track 0.00 -> 7.33 mm
- net GND: track 183.6 -> 187.0 mm, vias 81 -> 116
- net Net-(C32-Pad2): track 5.54 -> 3.23 mm
- net +3V3: track 49.8 -> 52.1 mm, vias 14 -> 17
- net TSENSE_2: track 44.7 -> 46.1 mm

Commit message: Gerbers added
Parts:
- moved J4 0.49 mm to (122.2, 126.7)
Connections:
- IC1 pad 114: Net-(IC1-Pad114) -> SD_CS
Routing:
- net SD_CS: track 0.00 -> 44.2 mm, vias 0 -> 2
- net SD_MOSI: track 48.8 -> 50.0 mm
- net GND: track 187.0 -> 185.9 mm, vias 116 -> 115
